Commit message: fixed package name issue

File: model/so101_new_calib.urdf (robot description, URDF)
Before this commit: robot so101_new_calib, 9 links, 8 joints
Links:
- link base_link: geometry collision mesh filename=package://so101_moveit2_description/model/assets/base_motor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; collision mesh filename=package://so101_moveit2_description/model/assets/base_so101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
- link gripper_link: geometry collision mesh filename=package://so101_moveit2_description/model/assets/sts3215_03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; collision mesh filename=package://so101_moveit2_description/model/assets/wrist_roll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
- link lower_arm_link: geometry collision mesh filename=package://so101_moveit2_description/model/assets/motor_hold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; collision mesh filename=package://so101_moveit2_description/model/assets/sts3215_03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
- link moving_jaw_so101_v1_link: geometry collision mesh filename=package://so101_moveit2_description/model/assets/moving_jaw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; visual mesh filename=package://so101_moveit2_description/model/assets/moving_jaw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
- link shoulder_link: geometry collision mesh filename=package://so101_moveit2_description/model/assets/motor_hold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; collision mesh filename=package://so101_moveit2_description/model/assets/rotation_p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
- link upper_arm_link: geometry collision mesh filename=package://so101_moveit2_description/model/assets/sts3215_03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; collision mesh filename=package://so101_moveit2_description/model/assets/upper_arm_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
- link wrist_link: geometry collision mesh filename=package://so101_moveit2_description/model/assets/sts3215_03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; collision mesh filename=package://so101_moveit2_description/model/assets/wrist_roll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

File: model/so101_new_calib.xacro (robot description, xacro)
@@ -29,5 +29,5 @@
       <origin xyz="-0.00636471 -9.94414e-05 -0.0024" rpy="1.5708 -1.67685e-15 1.5708"/>
       <geometry>
-        <mesh filename="file://$(find so101_moveit2)/model/assets/base_motor_holder_so101_v1.stl"/>
+        <mesh filename="file://$(find so101_moveit2_description)/model/assets/base_motor_holder_so101_v1.stl"/>
       </geometry>
       <material name="3d_printed"/>
@@ -36,5 +36,5 @@
       <origin xyz="-0.00636471 -9.94414e-05 -0.0024" rpy="1.5708 -1.67685e-15 1.5708"/>
       <geometry>
-        <mesh filename="file://$(find so101_moveit2)/model/assets/base_motor_holder_so101_v1.stl"/>
+        <mesh filename="file://$(find so101_moveit2_description)/model/assets/base_motor_holder_so101_v1.stl"/>
       </geometry>
     </collision>
@@ -43,5 +43,5 @@
       <origin xyz="-0.00636471 -8.97657e-09 -0.0024" rpy="1.5708 -2.78073e-29 1.5708"/>
       <geometry>
-        <mesh filename="file://$(find so101_moveit2)/model/assets/base_so101_v2.stl"/>
+        <mesh filename="file://$(find so101_moveit2_description)/model/assets/base_so101_v2.stl"/>
       </geometry>
       <material name="3d_printed"/>
@@ -50,5 +50,5 @@
       <origin xyz="-0.00636471 -8.97657e-09 -0.0024" rpy="1.5708 -2.78073e-29 1.5708"/>
       <geometry>
-        <mesh filename="file://$(find so101_moveit2)/model/assets/base_so101_v2.stl"/>
+        <mesh filename="file://$(find so101_moveit2_description)/model/assets/base_so101_v2.stl"/>
       </geometry>
     </collision>
@@ -57,5 +57,5 @@
       <origin xyz="0.0263353 -8.97657e-09 0.0437" rpy="-8.21148e-16 7.84513e-18 1.249e-15"/>
       <geometry>
-        <mesh filename="file://$(find so101_moveit2)/model/assets/sts3215_03a_v1.stl"/>
+        <mesh filename="file://$(find so101_moveit2_description)/model/assets/sts3215_03a_v1.stl"/>
       </geometry>
       <material name="sts3215"/>
@@ -64,5 +64,5 @@
       <origin xyz="0.0263353 -8.97657e-09 0.0437" rpy="-8.21148e-16 7.84513e-18 1.249e-15"/>
       <geometry>
-        <mesh filename="file://$(find so101_moveit2)/model/assets/sts3215_03a_v1.stl"/>
+        <mesh filename="file://$(find so101_moveit2_description)/model/assets/sts3215_03a_v1.stl"/>
       </geometry>
     </collision>
@@ -71,5 +71,5 @@
       <origin xyz="-0.0309827 -0.000199441 0.0474" rpy="1.5708 -1.35493e-14 1.5708"/>
       <geometry>
-        <mesh filename="file://$(find so101_moveit2)/model/assets/waveshare_mounting_plate_so101_v2.stl"/>
+        <mesh filename="file://$(find so101_moveit2_description)/model/assets/waveshare_mounting_plate_so101_v2.stl"/>
       </geometry>
       <material name="3d_printed"/>
@@ -78,5 +78,5 @@
       <origin xyz="-0.0309827 -0.000199441 0.0474" rpy="1.5708 -1.35493e-14 1.5708"/>
       <geometry>
-        <mesh filename="file://$(find so101_moveit2)/model/assets/waveshare_mounting_plate_so101_v2.stl"/>
+        <mesh filename="file://$(find so101_moveit2_description)/model/assets/waveshare_mounting_plate_so101_v2.stl"/>
       </geometry>
     </collision>
@@ -93,5 +93,5 @@
       <origin xyz="-0.0303992 0.000422241 -0.0417" rpy="1.5708 1.5708 0"/>
       <geometry>
-        <mesh filename="file://$(find so101_moveit2)/model/assets/sts3215_03a_v1.stl"/>
+        <mesh filename="file://$(find so101_moveit2_description)/model/assets/sts3215_03a_v1.stl"/>
       </geometry>
       <material name="sts3215"/>
@@ -100,5 +100,5 @@
       <origin xyz="-0.0303992 0.000422241 -0.0417" rpy="1.5708 1.5708 0"/>
       <geometry>
-        <mesh filename="file://$(find so101_moveit2)/model/assets/sts3215_03a_v1.stl"/>
+        <mesh filename="file://$(find so101_moveit2_description)/model/assets/sts3215_03a_v1.stl"/>
       </geometry>
     </collision>
@@ -107,5 +107,5 @@
       <origin xyz="-0.0675992 -0.000177759 0.0158499" rpy="1.5708 -1.5708 0"/>
       <geometry>
-        <mesh filename="file://$(find so101_moveit2)/model/assets/motor_holder_so101_base_v1.stl"/>
+        <mesh filename="file://$(find so101_moveit2_description)/model/assets/motor_holder_so101_base_v1.stl"/>
       </geometry>
       <material name="3d_printed"/>
@@ -114,5 +114,5 @@
       <origin xyz="-0.0675992 -0.000177759 0.0158499" rpy="1.5708 -1.5708 0"/>
       <geometry>
-        <mesh filename="file://$(find so101_moveit2)/model/assets/motor_holder_so101_base_v1.stl"/>
+        <mesh filename="file://$(find so101_moveit2_description)/model/assets/motor_holder_so101_base_v1.stl"/>
       </geometry>
     </collision>
@@ -121,5 +121,5 @@
       <origin xyz="0.0122008 2.22413e-05 0.0464" rpy="-1.5708 2.35221e-33 0"/>
       <geometry>
-        <mesh filename="file://$(find so101_moveit2)/model/assets/rotation_pitch_so101_v1.stl"/>
+        <mesh filename="file://$(find so101_moveit2_description)/model/assets/rotation_pitch_so101_v1.stl"/>
       </geometry>
       <material name="3d_printed"/>
@@ -128,5 +128,5 @@
       <origin xyz="0.0122008 2.22413e-05 0.0464" rpy="-1.5708 2.35221e-33 0"/>
       <geometry>
-        <mesh filename="file://$(find so101_moveit2)/model/assets/rotation_pitch_so101_v1.stl"/>
+        <mesh filename="file://$(find so101_moveit2_description)/model/assets/rotation_pitch_so101_v1.stl"/>
       </geometry>
     </collision>
@@ -143,5 +143,5 @@
       <origin xyz="-0.11257 -0.0155 0.0187" rpy="-3.14159 -5.27356e-16 -1.5708"/>
       <geometry>
-        <mesh filename="file://$(find so101_moveit2)/model/assets/sts3215_03a_v1.stl"/>
+        <mesh filename="file://$(find so101_moveit2_description)/model/assets/sts3215_03a_v1.stl"/>
       </geometry>
       <material name="sts3215"/>
@@ -150,5 +150,5 @@
       <origin xyz="-0.11257 -0.0155 0.0187" rpy="-3.14159 -5.27356e-16 -1.5708"/>
       <geometry>
-        <mesh filename="file://$(find so101_moveit2)/model/assets/sts3215_03a_v1.stl"/>
+        <mesh filename="file://$(find so101_moveit2_description)/model/assets/sts3215_03a_v1.stl"/>
       </geometry>
     </collision>
@@ -157,5 +157,5 @@
       <origin xyz="-0.065085 0.012 0.0182" rpy="3.14159 -0 -1.30911e-30"/>
       <geometry>
-        <mesh filename="file://$(find so101_moveit2)/model/assets/upper_arm_so101_v1.stl"/>
+        <mesh filename="file://$(find so101_moveit2_description)/model/assets/upper_arm_so101_v1.stl"/>
       </geometry>
       <material name="3d_printed"/>
@@ -164,5 +164,5 @@
       <origin xyz="-0.065085 0.012 0.0182" rpy="3.14159 -0 -1.30911e-30"/>
       <geometry>
-        <mesh filename="file://$(find so101_moveit2)/model/assets/upper_arm_so101_v1.stl"/>
+        <mesh filename="file://$(find so101_moveit2_description)/model/assets/upper_arm_so101_v1.stl"/>
       </geometry>
     </collision>
@@ -179,5 +179,5 @@
       <origin xyz="-0.0648499 -0.032 0.0182" rpy="3.14159 -0 6.67202e-31"/>
       <geometry>
-        <mesh filename="file://$(find so101_moveit2)/model/assets/under_arm_so101_v1.stl"/>
+        <mesh filename="file://$(find so101_moveit2_description)/model/assets/under_arm_so101_v1.stl"/>
       </geometry>
       <material name="3d_printed"/>
@@ -186,5 +186,5 @@
       <origin xyz="-0.0648499 -0.032 0.0182" rpy="3.14159 -0 6.67202e-31"/>
       <geometry>
-        <mesh filename="file://$(find so101_moveit2)/model/assets/under_arm_so101_v1.stl"/>
+        <mesh filename="file://$(find so101_moveit2_description)/model/assets/under_arm_so101_v1.stl"/>
       </geometry>
     </collision>
@@ -193,5 +193,5 @@
       <origin xyz="-0.0648499 -0.032 0.018" rpy="-3.14159 -2.55351e-15 -1.83387e-30"/>
       <geometry>
-        <mesh filename="file://$(find so101_moveit2)/model/assets/motor_holder_so101_wrist_v1.stl"/>
+        <mesh filename="file://$(find so101_moveit2_description)/model/assets/motor_holder_so101_wrist_v1.stl"/>
       </geometry>
       <material name="3d_printed"/>
@@ -200,5 +200,5 @@
       <origin xyz="-0.0648499 -0.032 0.018" rpy="-3.14159 -2.55351e-15 -1.83387e-30"/>
       <geometry>
-        <mesh filename="file://$(find so101_moveit2)/model/assets/motor_holder_so101_wrist_v1.stl"/>
+        <mesh filename="file://$(find so101_moveit2_description)/model/assets/motor_holder_so101_wrist_v1.stl"/>
       </geometry>
     </collision>
@@ -207,5 +207,5 @@
       <origin xyz="-0.1224 0.0052 0.0187" rpy="-3.14159 -7.88861e-31 -3.14159"/>
       <geometry>
-        <mesh filename="file://$(find so101_moveit2)/model/assets/sts3215_03a_v1.stl"/>
+        <mesh filename="file://$(find so101_moveit2_description)/model/assets/sts3215_03a_v1.stl"/>
       </geometry>
       <material name="sts3215"/>
@@ -214,5 +214,5 @@
       <origin xyz="-0.1224 0.0052 0.0187" rpy="-3.14159 -7.88861e-31 -3.14159"/>
       <geometry>
-        <mesh filename="file://$(find so101_moveit2)/model/assets/sts3215_03a_v1.stl"/>
+        <mesh filename="file://$(find so101_moveit2_description)/model/assets/sts3215_03a_v1.stl"/>
       </geometry>
     </collision>
@@ -229,5 +229,5 @@
       <origin xyz="8.32667e-17 -0.0424 0.0306" rpy="1.5708 1.5708 0"/>
       <geometry>
-        <mesh filename="file://$(find so101_moveit2)/model/assets/sts3215_03a_no_horn_v1.stl"/>
+        <mesh filename="file://$(find so101_moveit2_description)/model/assets/sts3215_03a_no_horn_v1.stl"/>
       </geometry>
       <material name="sts3215"/>
@@ -236,5 +236,5 @@
       <origin xyz="8.32667e-17 -0.0424 0.0306" rpy="1.5708 1.5708 0"/>
       <geometry>
-        <mesh filename="file://$(find so101_moveit2)/model/assets/sts3215_03a_no_horn_v1.stl"/>
+        <mesh filename="file://$(find so101_moveit2_description)/model/assets/sts3215_03a_no_horn_v1.stl"/>
       </geometry>
     </collision>
@@ -243,5 +243,5 @@
       <origin xyz="0 -0.028 0.0181" rpy="-1.5708 -1.5708 0"/>
       <geometry>
-        <mesh filename="file://$(find so101_moveit2)/model/assets/wrist_roll_pitch_so101_v2.stl"/>
+        <mesh filename="file://$(find so101_moveit2_description)/model/assets/wrist_roll_pitch_so101_v2.stl"/>
       </geometry>
       <material name="3d_printed"/>
@@ -250,5 +250,5 @@
       <origin xyz="0 -0.028 0.0181" rpy="-1.5708 -1.5708 0"/>
       <geometry>
-        <mesh filename="file://$(find so101_moveit2)/model/assets/wrist_roll_pitch_so101_v2.stl"/>
+        <mesh filename="file://$(find so101_moveit2_description)/model/assets/wrist_roll_pitch_so101_v2.stl"/>
       </geometry>
     </collision>
@@ -265,5 +265,5 @@
       <origin xyz="0.0077 0.0001 -0.0234" rpy="-1.5708 -5.19179e-17 -1.66533e-16"/>
       <geometry>
-        <mesh filename="file://$(find so101_moveit2)/model/assets/sts3215_03a_v1.stl"/>
+        <mesh filename="file://$(find so101_moveit2_description)/model/assets/sts3215_03a_v1.stl"/>
       </geometry>
       <material name="sts3215"/>
@@ -272,5 +272,5 @@
       <origin xyz="0.0077 0.0001 -0.0234" rpy="-1.5708 -5.19179e-17 -1.66533e-16"/>
       <geometry>
-        <mesh filename="file://$(find so101_moveit2)/model/assets/sts3215_03a_v1.stl"/>
+        <mesh filename="file://$(find so101_moveit2_description)/model/assets/sts3215_03a_v1.stl"/>
       </geometry>
     </collision>
@@ -279,5 +279,5 @@
       <origin xyz="8.32667e-17 -0.000218214 0.000949706" rpy="-3.14159 -5.55112e-17 0"/>
       <geometry>
-        <mesh filename="file://$(find so101_moveit2)/model/assets/wrist_roll_follower_so101_v1.stl"/>
+        <mesh filename="file://$(find so101_moveit2_description)/model/assets/wrist_roll_follower_so101_v1.stl"/>
       </geometry>
       <material name="3d_printed"/>
@@ -286,5 +286,5 @@
       <origin xyz="8.32667e-17 -0.000218214 0.000949706" rpy="-3.14159 -5.55112e-17 0"/>
       <geometry>
-        <mesh filename="file://$(find so101_moveit2)/model/assets/wrist_roll_follower_so101_v1.stl"/>
+        <mesh filename="file://$(find so101_moveit2_description)/model/assets/wrist_roll_follower_so101_v1.stl"/>
       </geometry>
     </collision>
@@ -316,5 +316,5 @@
       <origin xyz="-5.55112e-17 -5.55112e-17 0.0189" rpy="9.53145e-17 6.93889e-18 1.24077e-24"/>
       <geometry>
-        <mesh filename="file://$(find so101_moveit2)/model/assets/moving_jaw_so101_v1.stl"/>
+        <mesh filename="file://$(find so101_moveit2_description)/model/assets/moving_jaw_so101_v1.stl"/>
       </geometry>
       <material name="3d_printed"/>
@@ -323,5 +323,5 @@
       <origin xyz="-5.55112e-17 -5.55112e-17 0.0189" rpy="9.53145e-17 6.93889e-18 1.24077e-24"/>
       <geometry>
-        <mesh filename="file://$(find so101_moveit2)/model/assets/moving_jaw_so101_v1.stl"/>
+        <mesh filename="file://$(find so101_moveit2_description)/model/assets/moving_jaw_so101_v1.stl"/>
       </geometry>
     </collision>

Commit message: robot is now fixed to ground

File: model/so101_new_calib.urdf (robot description, URDF)
Before this commit: robot so101_new_calib, 9 links, 8 joints
Links:
- removed link root
- added link world
Joints:
- removed joint root_to_base
- added joint world_joint: type fixed, parent world, child base_link, origin xyz=0 0 0 rpy=0 0 0
